Commit message: feat: add compatible quadruped loco-manipulation tasks

File: source/robot_lab/data/Robots/unitree/go2_arx5/urdf/go2_arx5_finray_x85_z94.urdf (robot description, URDF)
Before this commit: robot go2arx5_finray, 41 links, 40 joints
Links:
- removed link FL_foot_target
- removed link FR_foot_target
- removed link RL_foot_target
- removed link RR_foot_target
Joints:
- removed joint FL_foot_target_joint
- removed joint FR_foot_target_joint
- removed joint RL_foot_target_joint
- removed joint RR_foot_target_joint
